File: complete project/EEE3088_design_project.kicad_pcb (KiCad board)
At the start: 2 copper layers, 40 parts, among them J1 Conn_01x02_Male, J2 Conn_01x10_Pin, J3 Conn_01x02_Male, U1 STM32F051C6Tx, U2 FT232RL, U3 AT24C256C-SSHL-T, U4 TP4056, U5 DW01A-G, U6 FS8205A_C908265, U7 HT75xx-1-SOT89, Y1 8MHz

Commit message: Latest update of PCB
Parts:
- removed U1: STM32F051C6Tx, STM32:STM32F051C6T6
- added J7: Conn_02x24_Counter_Clockwise, STM32:STM32F051C6T6, F.Cu at (144.8, 111.8)
Connections:
- net Net-(U1-NRST) renamed /Microcontroller Interface/NRST
Other:
- board outline added: 100.1 x 100.1 mm
