File: complete project/EEE3088_design_project.kicad_pcb (KiCad board)
At the start: 2 copper layers, 100.1 x 100.1 mm, 40 parts, among them J1 Conn_01x02_Male, J2 Conn_01x10_Pin, J3 Conn_01x02_Male, J7 Conn_02x24_Counter_Clockwise, U2 FT232RL, U3 AT24C256C-SSHL-T, U4 TP4056, U5 DW01A-G, U6 FS8205A_C908265, U7 HT75xx-1-SOT89, Y1 8MHz

Commit message: latest copy of PCB
Parts:
- added C13: 100n, Capacitor_SMD:C_0805_2012Metric, F.Cu at (117.9, 118.4)
- added J4: Conn_01x04_Pin, Connector_PinHeader_2.54mm:PinHeader_1x04_P2.54mm_Vertical, F.Cu at (115.3, 97.5)
- added J5: Conn_01x02_Pin, Connector_PinHeader_2.54mm:PinHeader_1x02_P2.54mm_Vertical, F.Cu at (122.4, 144.0)
- added J6: Conn_01x03_Pin, Connector_PinHeader_2.54mm:PinHeader_1x03_P2.54mm_Vertical, F.Cu at (163.1, 92.5)
- added J8: Conn_01x08_Pin, Connector_PinHeader_2.54mm:PinHeader_1x08_P2.54mm_Vertical, F.Cu at (106.2, 140.2)
- added R10: 4.7k, Resistor_SMD:R_0805_2012Metric_Pad1.20x1.40mm_HandSolder, F.Cu at (114.8, 104.6)
- added R11: 4.7k, Resistor_SMD:R_0805_2012Metric_Pad1.20x1.40mm_HandSolder, F.Cu at (118.9, 104.6)
- added R12: 5k, Resistor_SMD:R_0805_2012Metric_Pad1.20x1.40mm_HandSolder, F.Cu at (114.8, 135.1)
- added R8: 4K7, Resistor_SMD:R_0805_2012Metric_Pad1.20x1.40mm_HandSolder, F.Cu at (144.3, 113.3)
- added R9: 4K7, Resistor_SMD:R_0805_2012Metric_Pad1.20x1.40mm_HandSolder, F.Cu at (148.8, 113.3)
- added TH1: Thermistor, STM32:RES-TH_L12.5-W5.0-P7.50-D0.7, F.Cu at (114.8, 145.3)
- added TP10: Eprom SLC, TestPoint:TestPoint_THTPad_1.0x1.0mm_Drill0.5mm, F.Cu at (160.0, 118.4)
- added TP4: TestPoint, TestPoint:TestPoint_THTPad_1.0x1.0mm_Drill0.5mm, F.Cu at (116.8, 112.3)
- added TP5: Temp SDA, TestPoint:TestPoint_THTPad_1.0x1.0mm_Drill0.5mm, F.Cu at (108.2, 105.7)
- added TP6: Temp SLC, TestPoint:TestPoint_THTPad_1.0x1.0mm_Drill0.5mm, F.Cu at (108.2, 110.7)
- added TP7: V3.3, TestPoint:TestPoint_THTPad_1.0x1.0mm_Drill0.5mm, F.Cu at (122.4, 118.4)
- added TP8: Analog sens, TestPoint:TestPoint_THTPad_1.0x1.0mm_Drill0.5mm, F.Cu at (108.2, 116.8)
- added TP9: Eprom SDA, TestPoint:TestPoint_THTPad_1.0x1.0mm_Drill0.5mm, F.Cu at (160.0, 114.3)
- added U8: DHT22, STM32:SENSOR-TH_HAIGU_DHT22, F.Cu at (109.2, 93.7)
- J1, J3: footprint Connector_PinHeader_2.54mm:PinHeader_1x02_P2.54mm_Horizontal -> Connector_PinHeader_2.54mm:PinHeader_1x02_P2.54mm_Vertical
- J2: footprint Connector_PinHeader_2.54mm:PinHeader_1x10_P2.54mm_Horizontal -> Connector_PinHeader_2.54mm:PinHeader_1x10_P2.54mm_Vertical
- TP1: value TestPoint -> 5V
- TP2: value TestPoint -> GND
- moved C9 1.45 mm to (129.0, 151.4), turned to -90 degrees
Connections:
- C7 pad 2: +5V -> 5V
- C8 pad 2: +5V -> 5V
- C9 pad 1: GND -> 5V
- J2 pad 1: +5V -> 5V
- J3 pad 2: +5V -> 5V
- J7 pad 17: unconnected-(J7-Pin_17-Pad17) -> PA7
- J7 pad 44: unconnected-(J7-Pin_44-Pad44) -> Net-(J6-Pin_2)
- TP1 pad 1: +5V -> 5V
- U2 pad 20: +5V -> 5V
- USB1 pad 1: +5V -> 5V
- USB1 pad 6: unconnected-(USB1-SH1-Pad6) -> GND
- USB1 pad 7: unconnected-(USB1-SH2-Pad7) -> GND
- USB1 pad 8: unconnected-(USB1-SH3-Pad8) -> GND
- USB1 pad 9: unconnected-(USB1-SH4-Pad9) -> GND
Routing:
- net Vout3: track 240.2 -> 357.5 mm, vias 3 -> 9
- net 5V: track 0.00 -> 102.6 mm
- net GND: track 414.5 -> 512.0 mm, vias 0 -> 2
- net +5V: track 96.5 -> 0.00 mm
- net Temp_Sensor_SLC: track 8.68 -> 96.4 mm
- net Temp_Sensor_SDA: track 8.68 -> 85.4 mm
- net Analog temp sensor: track 19.9 -> 68.1 mm
- net PA2: track 0.00 -> 47.7 mm
- net PA0: track 0.00 -> 45.9 mm
- net PA7: track 0.00 -> 45.7 mm
- net PA1: track 0.00 -> 45.6 mm
- net PA6: track 0.00 -> 44.7 mm
- net PA5: track 0.00 -> 43.8 mm
- net PA4: track 0.00 -> 42.8 mm
- net PA3: track 0.00 -> 41.5 mm
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Other:
- board text added: "+"
- board text added: "-"
- board text added: "A0"
- board text added: "A1"
- board text added: "A2"
- board text added: "A3"
- board text added: "A4"
- board text added: "A5"
- board text added: "A6"
- board text added: "A7"
- board text added: "Group 32 Data logger"
- board text added: "Letsolo Leoma"
- board text added: "Matthew Rose-Innes"
- board text added: "Ntokozo Radebe"
- board text added: "Rev 1.0"
