File: complete project/EEE3088_design_project.kicad_pcb (KiCad board)
At the start: 2 copper layers, 100.1 x 100.1 mm, 59 parts, among them J1 Conn_01x02_Male, J2 Conn_01x10_Pin, J3 Conn_01x02_Male, J4 Conn_01x04_Pin, J5 Conn_01x02_Pin, J6 Conn_01x03_Pin, J7 Conn_02x24_Counter_Clockwise, J8 Conn_01x08_Pin, U2 FT232RL, U3 AT24C256C-SSHL-T, U4 TP4056, U5 DW01A-G, U6 FS8205A_C908265, U7 HT75xx-1-SOT89, U8 DHT22, Y1 8MHz

Commit message: corrected group details
Other:
- board text added: "Group 31 Data logger"
- board text removed: "Group 32 Data logger"
Changed lines of the file:
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@@
     (comment 1 "Added all components from power and microcontroller interface")
     (comment 2 "Added all sensors")
+    (comment 3 "Corrected group info")
   )
   (layers
@@
     (effects (font (size 1 1) (thickness 0.15)) (justify left bottom))
   )
-  (gr_text "Group 32 Data logger" (at 92.456 153.924 90) (layer "F.SilkS")
+  (gr_text "Group 31 Data logger" (at 92.456 153.924 90) (layer "F.SilkS")
     (effects (font (size 4 2) (thickness 0.4) bold) (justify left bottom))
   )

Commit message: update Justins comments
Parts:
- TP1: value 5V -> TestPoint
- moved R5 67.7 mm to (140.7, 147.8), turned to 90 degrees
Connections:
- R5 pad 1: /Power managment/POS_terminal -> Net-(U4-PROG)
- U4 pad 1: /Power managment/POS_terminal -> GND
- U4 pad 2: /Power managment/POS_terminal -> Net-(U4-PROG)
- U4 pad 3: /Power managment/POS_terminal -> GND
Routing:
- net GND: track 512.0 -> 492.4 mm
- net /Power managment/POS_terminal: track 167.7 -> 155.6 mm
- net Net-(U4-PROG): track 0.00 -> 3.78 mm
- added copper zone on F.Cu, net GND
