File: complete project/EEE3088_design_project.kicad_sch (KiCad schematic)
At the start: 0 parts

Commit message: latest copy of PCB
Other:
- added sheet Sensors (Sensors.kicad_sch)
Changed lines of the file:
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@@
 (kicad_sch (version 20230121) (generator eeschema)
   (paper "A4")
-  (sheet (at 26.67 26.67) (size 114.3 72.39) (fields_autoplaced)
+  (sheet (at 26.67 27.94) (size 114.3 72.39) (fields_autoplaced)
     (stroke (width 0.1524) (type solid))
     (fill (color 0 0 0 0.0000))
-    (property "Sheetname" "Power managment" (at 26.67 24.0934 0)
+    (property "Sheetname" "Power managment" (at 26.67 25.3634 0)
       (effects (font (size 5 5) bold) (justify left bottom))
     )
-    (property "Sheetfile" "power.kicad_sch" (at 26.67 99.6446 0)
+    (property "Sheetfile" "power.kicad_sch" (at 26.67 100.9146 0)
       (effects (font (size 1.27 1.27)) (justify left top))
     )
@@
       )
     )
+  )
+  (sheet (at 29.21 116.84) (size 115.57 54.61) (fields_autoplaced)
+    (stroke (width 0.1524) (type solid))
+    (fill (color 0 0 0 0.0000))
+    (property "Sheetname" "Sensors" (at 29.21 114.7634 0)
+      (effects (font (size 4 4) bold) (justify left bottom))
+    )
+    (property "Sheetfile" "Sensors.kicad_sch" (at 29.21 172.0346 0)
+      (effects (font (size 1.27 1.27)) (justify left top))
+    )
+    (instances
+      (project "EEE3088_design_project"
+        (path "/cce61722-d4ce-4f54-abf4-b299d0ab67e2" (page "4"))
+      )
+    )
