File: complete project/Microcontroller interface.kicad_sch (KiCad schematic)
At the start: 19 parts, among them J2 Conn_01x10_Pin, U1 STM32F051C6Tx, U2 FT232RL, U3 AT24C256C-SSHL-T, Y1 8MHz

Commit message: Latest update of PCB
Parts:
- removed U1: STM32F051C6Tx, STM32:STM32F051C6T6, symbol MCU_ST_STM32F0:STM32F051C6Tx
- added J7: Conn_02x24_Counter_Clockwise, STM32:STM32F051C6T6, symbol Connector_Generic:Conn_02x24_Counter_Clockwise
Connections:
- net +3.3V: now also J7.24 (Pin_24), J7.48 (Pin_48), J7.9 (Pin_9)
- net Analog temp sensor: now also J7.18 (Pin_18)
- net Eprom_SDA: now also J7.36 (Pin_36)
- net Eprom_SLC: now also J7.35 (Pin_35)
- net GND: now also USB1.6 (SH1), USB1.7 (SH2), USB1.8 (SH3), USB1.9 (SH4), J7.23 (Pin_23), J7.47 (Pin_47), J7.8 (Pin_8)
- net PA0: now also J7.10 (Pin_10)
- net PA1: now also J7.11 (Pin_11)
- net PA11: now also J7.32 (Pin_32)
- net PA12: now also J7.33 (Pin_33)
- net PA13: now also J7.34 (Pin_34)
- net PA14: now also J7.37 (Pin_37)
- net PA15: now also J7.38 (Pin_38)
- net PA2: now also J7.12 (Pin_12)
- net PA3: now also J7.13 (Pin_13)
- net PA4: now also J7.14 (Pin_14)
- net PA5: now also J7.15 (Pin_15)
- net PA6: now also J7.16 (Pin_16)
- net PA7: now also J7.17 (Pin_17)
- net PA8: now also J7.29 (Pin_29)
- net PB1: now also J7.19 (Pin_19)
- net PB12: now also J7.25 (Pin_25)
- net PB13: now also J7.26 (Pin_26)
- net PB14: now also J7.27 (Pin_27)
- net PB15: now also J7.28 (Pin_28)
- net PB2: now also J7.20 (Pin_20)
- net PB3: now also J7.39 (Pin_39)
- net PB4: now also J7.40 (Pin_40)
- net PB5: now also J7.41 (Pin_41)
- net PB6: now also J7.42 (Pin_42)
- net PB7: now also J7.43 (Pin_43)
- net PB8: now also J7.45 (Pin_45)
- net PB9: now also J7.46 (Pin_46)
- net RX: now also J7.30 (Pin_30)
- net TX: now also J7.31 (Pin_31)
- net Temp_Sensor_SDA: now also J7.22 (Pin_22)
- net Temp_Sensor_SLC: now also J7.21 (Pin_21)
- net at C4.2, Y1.1: now also J7.5 (Pin_5)
- net at C3.2, Y1.2: now also J7.6 (Pin_6)
- net NRST: now reaches C6.2, S1.4
- net NRST: now also J7.7 (Pin_7)
- net +5V renamed 5V
- net 5V: no longer USB1.1 (VBUS)
- new net V5: USB1.1 (VBUS)
- no-connect marks 20 -> 24
Other:
- note added: "Updated STM32 to be a header and not the actual STM32 IC. Added name to the Schematic"
- company: (none) -> Matthew Rose-Innes
- title: (none) -> EEE3088F design project microcontroller schematic

Commit message: latest copy of PCB
Parts:
- added J6: Conn_01x03_Pin, Connector_PinHeader_2.54mm:PinHeader_1x03_P2.54mm_Vertical, symbol Connector:Conn_01x03_Pin
- added J8: Conn_01x08_Pin, Connector_PinHeader_2.54mm:PinHeader_1x08_P2.54mm_Vertical, symbol Connector:Conn_01x08_Pin
- added R2 (x2): 4K7, Resistor_SMD:R_0805_2012Metric_Pad1.20x1.40mm_HandSolder, symbol Device:R
- added TP4: Eprom SLC, TestPoint:TestPoint_THTPad_1.0x1.0mm_Drill0.5mm, symbol Connector:TestPoint
- added TP4: Eprom SDA, TestPoint:TestPoint_THTPad_1.0x1.0mm_Drill0.5mm, symbol Connector:TestPoint
- J2: footprint Connector_PinHeader_2.54mm:PinHeader_1x10_P2.54mm_Horizontal -> Connector_PinHeader_2.54mm:PinHeader_1x10_P2.54mm_Vertical
Connections:
- net +3.3V: now also J6.1 (Pin_1), R2.2, R2.2
- net Eprom_SDA: now also R2.1, TP4.1
- net Eprom_SLC: now also R2.1, TP4.1
- net GND: now also J6.3 (Pin_3)
- net PA0: now also J8.8 (Pin_8)
- net PA1: now also J8.7 (Pin_7)
- net PA2: now also J8.6 (Pin_6)
- net PA3: now also J8.5 (Pin_5)
- net PA4: now also J8.4 (Pin_4)
- net PA5: now also J8.3 (Pin_3)
- net PA6: now also J8.2 (Pin_2)
- net PA7: now also J8.1 (Pin_1)
- net at J7.44 (Pin_44): now also J6.2 (Pin_2)
- no-connect marks 24 -> 23

Commit message: update Justins comments
Parts:
- renumbered TP4 to TP7
Changed lines of the file:
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@@
   (symbol (lib_id "Connector:TestPoint") (at 232.41 114.3 180) (unit 1)
     (in_bom yes) (on_board yes) (dnp no)
-    (property "Reference" "TP4" (at 234.95 116.967 0)
+    (property "Reference" "TP7" (at 234.95 116.967 0)
       (effects (font (size 1.27 1.27)) (justify right))
     )
@@
   (symbol (lib_id "Connector:TestPoint") (at 242.57 93.98 0) (unit 1)
     (in_bom yes) (on_board yes) (dnp no) (fields_autoplaced)
-    (property "Reference" "TP4" (at 245.11 90.043 0)
+    (property "Reference" "TP7" (at 245.11 90.043 0)
       (effects (font (size 1.27 1.27)) (justify left))
     )
