File: complete project/Sensors.kicad_sch (KiCad schematic)
At the start: 13 parts, among them J4 Conn_01x04_Pin, J5 Conn_01x02_Pin, U2 DHT22

Commit message: update Justins comments
Parts:
- renumbered C1 to C13, R1 to R10, R2 to R11, R3 to R12, TP1 to TP4, TP2 to TP5, TP3 to TP6, TP4 to TP7, TP5 to TP8, U2 to U8
Changed lines of the file:
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@@
   (symbol (lib_id "Connector:TestPoint") (at 95.25 127 180) (unit 1)
     (in_bom yes) (on_board yes) (dnp no) (fields_autoplaced)
-    (property "Reference" "TP5" (at 97.79 129.667 0)
+    (property "Reference" "TP8" (at 97.79 129.667 0)
       (effects (font (size 1.27 1.27)) (justify right))
     )
@@
   (symbol (lib_id "Device:R_Small") (at 87.63 120.65 0) (unit 1)
     (in_bom yes) (on_board yes) (dnp no) (fields_autoplaced)
-    (property "Reference" "R3" (at 90.17 120.015 0)
+    (property "Reference" "R12" (at 90.17 120.015 0)
       (effects (font (size 1.27 1.27)) (justify left))
     )
@@
   (symbol (lib_id "Device:C_Small") (at 64.77 53.34 0) (unit 1)
     (in_bom yes) (on_board yes) (dnp no) (fields_autoplaced)
-    (property "Reference" "C1" (at 67.31 52.7113 0)
+    (property "Reference" "C13" (at 67.31 52.7113 0)
       (effects (font (size 1.27 1.27)) (justify left))
     )
@@
   (symbol (lib_id "Connector:TestPoint") (at 116.84 59.69 180) (unit 1)
     (in_bom yes) (on_board yes) (dnp no) (fields_autoplaced)
-    (property "Reference" "TP3" (at 119.38 62.357 0)
+    (property "Reference" "TP6" (at 119.38 62.357 0)
       (effects (font (size 1.27 1.27)) (justify right))
     )
@@
   (symbol (lib_id "Connector:TestPoint") (at 87.63 115.57 270) (unit 1)
     (in_bom yes) (on_board yes) (dnp no) (fields_autoplaced)
-    (property "Reference" "TP4" (at 92.71 114.935 90)
+    (property "Reference" "TP7" (at 92.71 114.935 90)
       (effects (font (size 1.27 1.27)) (justify left))
     )
@@
   (symbol (lib_id "Device:R_Small") (at 120.65 54.61 0) (unit 1)
     (in_bom yes) (on_board yes) (dnp no) (fields_autoplaced)
-    (property "Reference" "R2" (at 123.19 53.975 0)
+    (property "Reference" "R11" (at 123.19 53.975 0)
       (effects (font (size 1.27 1.27)) (justify left))
     )
@@
   (symbol (lib_id "power:GND") (at 87.63 143.51 0) (unit 1)
     (in_bom yes) (on_board yes) (dnp no) (fields_autoplaced)
-    (property "Reference" "#PWR02" (at 87.63 149.86 0)
+    (property "Reference" "#PWR0105" (at 87.63 149.86 0)
       (effects (font (size 1.27 1.27)) hide)
     )
@@
   (symbol (lib_id "Connector:TestPoint") (at 67.31 45.72 0) (unit 1)
     (in_bom yes) (on_board yes) (dnp no) (fields_autoplaced)
-    (property "Reference" "TP1" (at 69.85 41.783 0)
+    (property "Reference" "TP4" (at 69.85 41.783 0)
       (effects (font (size 1.27 1.27)) (justify left))
     )
@@
   (symbol (lib_name "DHT22_1") (lib_id "DHT22:DHT22") (at 78.74 64.77 0) (unit 1)
     (in_bom yes) (on_board yes) (dnp no) (fields_autoplaced)
-    (property "Reference" "U2" (at 83.82 48.26 0)
+    (property "Reference" "U8" (at 83.82 48.26 0)
       (effects (font (size 1.27 1.27)))
     )
@@
   (symbol (lib_id "power:GND") (at 182.88 63.5 0) (unit 1)
     (in_bom yes) (on_board yes) (dnp no) (fields_autoplaced)
-    (property "Reference" "#PWR01" (at 182.88 69.85 0)
+    (property "Reference" "#PWR06" (at 182.88 69.85 0)
       (effects (font (size 1.27 1.27)) hide)
     )
@@
   (symbol (lib_id "power:GND") (at 99.06 67.31 0) (unit 1)
     (in_bom yes) (on_board yes) (dnp no) (fields_autoplaced)
-    (property "Reference" "#PWR01" (at 99.06 73.66 0)
+    (property "Reference" "#PWR0102" (at 99.06 73.66 0)
       (effects (font (size 1.27 1.27)) hide)
     )
@@
   (symbol (lib_id "Device:R_Small") (at 107.95 52.07 0) (unit 1)
     (in_bom yes) (on_board yes) (dnp no) (fields_autoplaced)
-    (property "Reference" "R1" (at 110.49 51.435 0)
+    (property "Reference" "R10" (at 110.49 51.435 0)
       (effects (font (size 1.27 1.27)) (justify left))
     )
@@
   (symbol (lib_id "Connector:TestPoint") (at 102.87 57.15 0) (unit 1)
     (in_bom yes) (on_board yes) (dnp no)
-    (property "Reference" "TP2" (at 99.06 55.88 0)
-      (effects (font (size 1.27 1.27)) (justify left))
-    )
+    (property "Reference" "TP5" (at 99.06 55.88 0)
+      (effects (font (size 1.27 1.27)) (justify left))
+    )
