File: complete project/power.kicad_sch (KiCad schematic)
At the start: 21 parts, among them J1 Conn_01x02_Male, J3 Conn_01x02_Male, U1 HT75xx-1-SOT89, U3 DW01A-G, U4 TP4056, U6 FS8205A_C908265

Commit message: Latest update of PCB
Connections:
- net +5V renamed V5
Changed lines of the file:
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@@
   (junction (at 99.06 80.01) (diameter 0) (color 0 0 0 0)
   )
+  (junction (at 125.73 48.26) (diameter 0) (color 0 0 0 0)
+  )
+  (junction (at 68.58 125.73) (diameter 0) (color 0 0 0 0)
+  )
+  (junction (at 106.68 48.26) (diameter 0) (color 0 0 0 0)
+  )
+  (junction (at 186.69 34.29) (diameter 0) (color 0 0 0 0)
+  )
+  (junction (at 208.28 80.01) (diameter 0) (color 0 0 0 0)
+  )
+  (junction (at 264.16 34.29) (diameter 0) (color 0 0 0 0)
+  )
   (junction (at 73.66 125.73) (diameter 0) (color 0 0 0 0)
-  )
-  (junction (at 125.73 48.26) (diameter 0) (color 0 0 0 0)
-  )
-  (junction (at 68.58 125.73) (diameter 0) (color 0 0 0 0)
-  )
-  (junction (at 106.68 48.26) (diameter 0) (color 0 0 0 0)
-  )
-  (junction (at 186.69 34.29) (diameter 0) (color 0 0 0 0)
-  )
-  (junction (at 208.28 80.01) (diameter 0) (color 0 0 0 0)
-  )
-  (junction (at 264.16 34.29) (diameter 0) (color 0 0 0 0)
   )
   (junction (at 128.27 80.01) (diameter 0) (color 0 0 0 0)
@@
     (stroke (width 0) (type default))
   )
-  (wire (pts (xy 73.66 125.73) (xy 76.2 125.73))
-    (stroke (width 0) (type default))
-  )
   (polyline (pts (xy 74.93 85.09) (xy 12.7 85.09))
     (stroke (width 0) (type default))
@@
   )
   (wire (pts (xy 128.27 25.4) (xy 186.69 25.4))
+    (stroke (width 0) (type default))
+  )
+  (wire (pts (xy 73.66 125.73) (xy 81.28 125.73))
     (stroke (width 0) (type default))
   )
@@
     (effects (font (size 1.27 1.27)) (justify left bottom))
   )
+  (label "Vout" (at 81.28 125.73 0) (fields_autoplaced)
+    (effects (font (size 1.27 1.27) bold) (justify left bottom))
+  )
   (label "Vout" (at 35.56 160.02 0) (fields_autoplaced)
     (effects (font (size 1.27 1.27)) (justify left bottom))
@@
     (effects (font (size 1.27 1.27)) (justify left bottom))
   )
-  (global_label "Vout3" (shape input) (at 77.47 116.84 0) (fields_autoplaced)
+  (global_label "Vout3" (shape output) (at 77.47 116.84 0) (fields_autoplaced)
     (effects (font (size 1.27 1.27)) (justify left))
     (property "Intersheetrefs" "${INTERSHEET_REFS}" (at 85.6976 116.84 0)
@@
     )
   )
-  (hierarchical_label "Vout" (shape input) (at 76.2 125.73 0) (fields_autoplaced)
-    (effects (font (size 1.27 1.27)) (justify left))
+  (global_label "V5" (shape input) (at 40.64 44.45 0) (fields_autoplaced)
+    (effects (font (size 1.27 1.27) bold) (justify left))
+    (property "Intersheetrefs" "${INTERSHEET_REFS}" (at 46.2723 44.45 0)
+      (effects (font (size 1.27 1.27)) (justify left) hide)
+    )
   )
   (symbol (lib_id "Regulator_Linear:HT75xx-1-SOT89") (at 54.61 128.27 0) (unit 1)
@@
         )
       )
-    )
-  )
-  (symbol (lib_id "power:+5V") (at 40.64 44.45 0) (unit 1)
-    (in_bom yes) (on_board yes) (dnp no)
-    (property "Reference" "#PWR06" (at 40.64 48.26 0)
-      (effects (font (size 1.27 1.27)) hide)
-    )
-    (property "Value" "+5V" (at 41.021 40.0558 0)
-      (effects (font (size 1.27 1.27)))
-    )
-    (property "Footprint" "" (at 40.64 44.45 0)
-      (effects (font (size 1.27 1.27)) hide)
-    )
-    (property "Datasheet" "" (at 40.64 44.45 0)
-      (effects (font (size 1.27 1.27)) hide)
-    )
-    (pin "1")
-    (instances
-      (project "SCHEMATICS"
-        (path "/a304c04d-6ae8-4b1e-9bcf-1dfdad79039c"
-          (reference "#PWR06") (unit 1)
-        )
-      )
-      (project "EEE3088_design_project"
-        (path "/cce61722-d4ce-4f54-abf4-b299d0ab67e2/12efe97a-1471-4a68-90a7-acf5ba080499"
-          (reference "#PWR06") (unit 1)
-        )
-      )

Commit message: latest copy of PCB
Parts:
- J1, J3: footprint Connector_PinHeader_2.54mm:PinHeader_1x02_P2.54mm_Horizontal -> Connector_PinHeader_2.54mm:PinHeader_1x02_P2.54mm_Vertical
- TP2: value TestPoint -> GND
Connections:
- net GND: no longer C3.1, D1.2 (A), D2.2 (A), J3.1 (Pin_1), U4.4 (VCC), U4.8 (CE)
- new net: C3.1, D1.2 (A), D2.2 (A), J3.1 (Pin_1), U4.4 (VCC), U4.8 (CE)
Changed lines of the file:
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@@
 (kicad_sch (version 20230121) (generator eeschema)
   (paper "A4")
+  (junction (at 99.06 48.26) (diameter 0) (color 0 0 0 0)
+  )
   (junction (at 99.06 80.01) (diameter 0) (color 0 0 0 0)
   )
-  (junction (at 125.73 48.26) (diameter 0) (color 0 0 0 0)
-  )
   (junction (at 68.58 125.73) (diameter 0) (color 0 0 0 0)
   )
@@
   (junction (at 208.28 67.31) (diameter 0) (color 0 0 0 0)
   )
-  (junction (at 125.73 80.01) (diameter 0) (color 0 0 0 0)
-  )
   (junction (at 154.94 72.39) (diameter 0) (color 0 0 0 0)
-  )
-  (junction (at 99.06 48.26) (diameter 0) (color 0 0 0 0)
   )
   (junction (at 38.1 125.73) (diameter 0) (color 0 0 0 0)
@@
     (stroke (width 0) (type default))
   )
-  (wire (pts (xy 99.06 80.01) (xy 125.73 80.01))
-    (stroke (width 0) (type default))
-  )
   (polyline (pts (xy 283.21 114.3) (xy 283.21 24.13))
     (stroke (width 0) (type default))
@@
     (stroke (width 0) (type default))
   )
+  (wire (pts (xy 99.06 48.26) (xy 99.06 57.15))
+    (stroke (width 0) (type default))
+  )
   (wire (pts (xy 106.68 48.26) (xy 116.84 48.26))
     (stroke (width 0) (type default))
@@
     (stroke (width 0) (type default))
   )
-  (wire (pts (xy 125.73 80.01) (xy 128.27 80.01))
+  (wire (pts (xy 99.06 80.01) (xy 128.27 80.01))
     (stroke (width 0) (type default))
   )
@@
     (stroke (width 0) (type default))
   )
+  (polyline (pts (xy 193.04 24.13) (xy 77.47 24.13))
+    (stroke (width 0) (type default))
+  )
+  (wire (pts (xy 40.64 44.45) (xy 40.64 48.26))
+    (stroke (width 0) (type default))
+  )
+  (polyline (pts (xy 193.04 54.61) (xy 283.21 54.61))
+    (stroke (width 0) (type default))
+  )
+  (wire (pts (xy 260.35 68.58) (xy 260.35 44.45))
+    (stroke (width 0) (type default))
+  )
+  (wire (pts (xy 27.94 80.01) (xy 99.06 80.01))
+    (stroke (width 0) (type default))
+  )
+  (wire (pts (xy 208.28 67.31) (xy 217.17 67.31))
+    (stroke (width 0) (type default))
+  )
+  (polyline (pts (xy 74.93 85.09) (xy 12.7 85.09))
+    (stroke (width 0) (type default))
+  )
+  (polyline (pts (xy 13.97 91.44) (xy 102.87 91.44))
+    (stroke (width 0) (type default))
+  )
+  (wire (pts (xy 252.73 46.99) (xy 264.16 46.99))
+    (stroke (width 0) (type default))
+  )
+  (wire (pts (xy 38.1 125.73) (xy 41.91 125.73))
+    (stroke (width 0) (type default))
+  )
+  (wire (pts (xy 264.16 34.29) (xy 264.16 46.99))
+    (stroke (width 0) (type default))
+  )
+  (wire (pts (xy 260.35 44.45) (xy 241.3 44.45))
+    (stroke (width 0) (type default))
+  )
+  (wire (pts (xy 116.84 48.26) (xy 125.73 48.26))
+    (stroke (width 0) (type default))
+  )
+  (wire (pts (xy 40.64 48.26) (xy 54.61 48.26))
+    (stroke (width 0) (type default))
+  )
+  (polyline (pts (xy 193.04 114.3) (xy 283.21 114.3))
+    (stroke (width 0) (type default))
+  )
+  (polyline (pts (xy 102.87 91.44) (xy 102.87 198.12))
+    (stroke (width 0) (type default))
+  )
+  (wire (pts (xy 154.94 69.85) (xy 154.94 72.39))
+    (stroke (width 0) (type default))
+  )
+  (wire (pts (xy 54.61 133.35) (xy 54.61 139.7))
+    (stroke (width 0) (type default))
+  )
+  (wire (pts (xy 41.91 125.73) (xy 46.99 125.73))
+    (stroke (width 0) (type default))
+  )
+  (wire (pts (xy 264.16 46.99) (xy 271.78 46.99))
+    (stroke (width 0) (type default))
+  )
+  (wire (pts (xy 199.39 34.29) (xy 264.16 34.29))
+    (stroke (width 0) (type default))
+  )
+  (wire (pts (xy 128.27 72.39) (xy 128.27 80.01))
+    (stroke (width 0) (type default))
+  )
+  (wire (pts (xy 106.68 76.2) (xy 137.16 76.2))
+    (stroke (width 0) (type default))
+  )
+  (wire (pts (xy 215.9 46.99) (xy 208.28 46.99))
+    (stroke (width 0) (type default))
+  )
+  (wire (pts (xy 128.27 25.4) (xy 186.69 25.4))
+    (stroke (width 0) (type default))
+  )
+  (wire (pts (xy 73.66 125.73) (xy 81.28 125.73))
+    (stroke (width 0) (type default))
+  )
   (wire (pts (xy 99.06 48.26) (xy 106.68 48.26))
     (stroke (width 0) (type default))
   )
-  (polyline (pts (xy 193.04 24.13) (xy 77.47 24.13))
-    (stroke (width 0) (type default))
-  )
-  (wire (pts (xy 40.64 44.45) (xy 40.64 48.26))
-    (stroke (width 0) (type default))
-  )
-  (polyline (pts (xy 193.04 54.61) (xy 283.21 54.61))
-    (stroke (width 0) (type default))
-  )
-  (wire (pts (xy 260.35 68.58) (xy 260.35 44.45))
-    (stroke (width 0) (type default))
-  )
-  (wire (pts (xy 27.94 80.01) (xy 99.06 80.01))
-    (stroke (width 0) (type default))
-  )
-  (wire (pts (xy 208.28 67.31) (xy 217.17 67.31))
-    (stroke (width 0) (type default))
-  )
-  (polyline (pts (xy 74.93 85.09) (xy 12.7 85.09))
-    (stroke (width 0) (type default))
-  )
-  (polyline (pts (xy 13.97 91.44) (xy 102.87 91.44))
-    (stroke (width 0) (type default))
-  )
-  (wire (pts (xy 252.73 46.99) (xy 264.16 46.99))
-    (stroke (width 0) (type default))
-  )
-  (wire (pts (xy 38.1 125.73) (xy 41.91 125.73))
-    (stroke (width 0) (type default))
-  )
-  (wire (pts (xy 264.16 34.29) (xy 264.16 46.99))
-    (stroke (width 0) (type default))
-  )
-  (wire (pts (xy 99.06 48.26) (xy 99.06 57.15))
-    (stroke (width 0) (type default))
-  )
-  (wire (pts (xy 260.35 44.45) (xy 241.3 44.45))
-    (stroke (width 0) (type default))
-  )
-  (wire (pts (xy 116.84 48.26) (xy 125.73 48.26))
-    (stroke (width 0) (type default))
-  )
-  (wire (pts (xy 40.64 48.26) (xy 54.61 48.26))
-    (stroke (width 0) (type default))
-  )
-  (polyline (pts (xy 193.04 114.3) (xy 283.21 114.3))
-    (stroke (width 0) (type default))
-  )
-  (polyline (pts (xy 102.87 91.44) (xy 102.87 198.12))
-    (stroke (width 0) (type default))
-  )
-  (wire (pts (xy 154.94 69.85) (xy 154.94 72.39))
-    (stroke (width 0) (type default))
-  )
-  (wire (pts (xy 54.61 133.35) (xy 54.61 139.7))
-    (stroke (width 0) (type default))
-  )
-  (wire (pts (xy 41.91 125.73) (xy 46.99 125.73))
-    (stroke (width 0) (type default))
-  )
-  (wire (pts (xy 264.16 46.99) (xy 271.78 46.99))
-    (stroke (width 0) (type default))
-  )
-  (wire (pts (xy 199.39 34.29) (xy 264.16 34.29))
-    (stroke (width 0) (type default))
-  )
-  (wire (pts (xy 128.27 72.39) (xy 128.27 80.01))
-    (stroke (width 0) (type default))
-  )
-  (wire (pts (xy 106.68 76.2) (xy 137.16 76.2))
-    (stroke (width 0) (type default))
-  )
-  (wire (pts (xy 215.9 46.99) (xy 208.28 46.99))
-    (stroke (width 0) (type default))
-  )
-  (wire (pts (xy 128.27 25.4) (xy 186.69 25.4))
-    (stroke (width 0) (type default))
-  )
-  (wire (pts (xy 73.66 125.73) (xy 81.28 125.73))
-    (stroke (width 0) (type default))
-  )
   (wire (pts (xy 38.1 125.73) (xy 38.1 132.08))
     (stroke (width 0) (type default))
@@
     (stroke (width 0) (type default))
   )
-  (wire (pts (xy 125.73 48.26) (xy 125.73 80.01))
-    (stroke (width 0) (type default))
-  )
   (polyline (pts (xy 283.21 24.13) (xy 193.04 24.13))
     (stroke (width 0) (type default))
@@
     (stroke (width 0) (type default))
   )
-  (wire (pts (xy 33.02 125.73) (xy 38.1 125.73))
+  (wire (pts (xy 21.59 125.73) (xy 38.1 125.73))
     (stroke (width 0) (type default))
   )
@@
     (effects (font (size 1.27 1.27)) (justify left bottom))
   )
-  (label "POS_terminal" (at 33.02 125.73 0) (fields_autoplaced)
+  (label "POS_terminal" (at 21.59 125.73 0) (fields_autoplaced)
     (effects (font (size 1.27 1.27)) (justify left bottom))
   )
@@
       (effects (font (size 1.27 1.27)))
     )
-    (property "Footprint" "Connector_PinHeader_2.54mm:PinHeader_1x02_P2.54mm_Horizontal" (at 30.48 157.48 0)
+    (property "Footprint" "Connector_PinHeader_2.54mm:PinHeader_1x02_P2.54mm_Vertical" (at 30.48 157.48 0)
       (effects (font (size 1.27 1.27)) hide)
     )
@@
       (effects (font (size 1.27 1.27)) (justify left) hide)
     )
-    (property "Value" "TestPoint" (at 17.9832 73.1012 0)
+    (property "Value" "GND" (at 17.9832 73.1012 0)
       (effects (font (size 1.27 1.27)) (justify left))
     )
@@
       (effects (font (size 1.27 1.27)) (justify left))
     )
-    (property "Footprint" "Connector_PinHeader_2.54mm:PinHeader_1x02_P2.54mm_Horizontal" (at 85.09 43.18 0)
-      (effects (font (size 1.27 1.27)) hide)
-    )
+    (property "Footprint" "Connector_PinHeader_2.54mm:PinHeader_1x02_P2.54mm_Vertical" (at 85.09 43.18 0)
+      (effects (font (size 1.27 1.27)) hide)
+    )

Commit message: update Justins comments
Connections:
- net GND: now also U4.1 (TEMP), U4.3 (GND)
- net POS_terminal: no longer R5.1, U4.1 (TEMP), U4.2 (PROG), U4.3 (GND)
- new net: R5.1, U4.2 (PROG)
Other:
- moved on the sheet: R5
Changed lines of the file:
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@@
   (junction (at 99.06 80.01) (diameter 0) (color 0 0 0 0)
   )
+  (junction (at 154.94 72.39) (diameter 0) (color 0 0 0 0)
+  )
   (junction (at 68.58 125.73) (diameter 0) (color 0 0 0 0)
   )
   (junction (at 106.68 48.26) (diameter 0) (color 0 0 0 0)
   )
-  (junction (at 186.69 34.29) (diameter 0) (color 0 0 0 0)
+  (junction (at 170.18 72.39) (diameter 0) (color 0 0 0 0)
   )
   (junction (at 208.28 80.01) (diameter 0) (color 0 0 0 0)
@@
   (junction (at 73.66 125.73) (diameter 0) (color 0 0 0 0)
   )
-  (junction (at 128.27 80.01) (diameter 0) (color 0 0 0 0)
-  )
-  (junction (at 170.18 57.15) (diameter 0) (color 0 0 0 0)
-  )
   (junction (at 116.84 48.26) (diameter 0) (color 0 0 0 0)
   )
+  (junction (at 154.94 80.01) (diameter 0) (color 0 0 0 0)
+  )
   (junction (at 41.91 125.73) (diameter 0) (color 0 0 0 0)
   )
   (junction (at 264.16 46.99) (diameter 0) (color 0 0 0 0)
   )
-  (junction (at 128.27 60.96) (diameter 0) (color 0 0 0 0)
-  )
   (junction (at 54.61 48.26) (diameter 0) (color 0 0 0 0)
   )
@@
   )
   (junction (at 208.28 67.31) (diameter 0) (color 0 0 0 0)
-  )
-  (junction (at 154.94 72.39) (diameter 0) (color 0 0 0 0)
   )
   (junction (at 38.1 125.73) (diameter 0) (color 0 0 0 0)
@@
     (stroke (width 0) (type default))
   )
-  (wire (pts (xy 128.27 60.96) (xy 128.27 64.77))
-    (stroke (width 0) (type default))
-  )
   (wire (pts (xy 54.61 48.26) (xy 54.61 45.72))
     (stroke (width 0) (type default))
@@
     (stroke (width 0) (type default))
   )
-  (wire (pts (xy 135.89 72.39) (xy 135.89 60.96))
-    (stroke (width 0) (type default))
-  )
-  (wire (pts (xy 186.69 25.4) (xy 186.69 34.29))
-    (stroke (width 0) (type default))
-  )
-  (wire (pts (xy 170.18 57.15) (xy 170.18 72.39))
-    (stroke (width 0) (type default))
-  )
   (wire (pts (xy 99.06 69.85) (xy 99.06 80.01))
     (stroke (width 0) (type default))
@@
     (stroke (width 0) (type default))
   )
-  (wire (pts (xy 154.94 72.39) (xy 135.89 72.39))
-    (stroke (width 0) (type default))
-  )
   (wire (pts (xy 199.39 39.37) (xy 199.39 34.29))
     (stroke (width 0) (type default))
@@
     (stroke (width 0) (type default))
   )
+  (wire (pts (xy 154.94 80.01) (xy 208.28 80.01))
+    (stroke (width 0) (type default))
+  )
   (wire (pts (xy 186.69 34.29) (xy 186.69 39.37))
     (stroke (width 0) (type default))
@@
     (stroke (width 0) (type default))
   )
-  (wire (pts (xy 135.89 60.96) (xy 128.27 60.96))
-    (stroke (width 0) (type default))
-  )
   (wire (pts (xy 99.06 48.26) (xy 99.06 57.15))
     (stroke (width 0) (type default))
@@
     (stroke (width 0) (type default))
   )
-  (wire (pts (xy 99.06 80.01) (xy 128.27 80.01))
-    (stroke (width 0) (type default))
-  )
-  (wire (pts (xy 170.18 49.53) (xy 170.18 57.15))
-    (stroke (width 0) (type default))
-  )
   (wire (pts (xy 125.73 34.29) (xy 125.73 41.91))
     (stroke (width 0) (type default))
@@
     (stroke (width 0) (type default))
   )
+  (wire (pts (xy 170.18 57.15) (xy 170.18 60.96))
+    (stroke (width 0) (type default))
+  )
   (polyline (pts (xy 193.04 24.13) (xy 77.47 24.13))
     (stroke (width 0) (type default))
@@
     (stroke (width 0) (type default))
   )
+  (wire (pts (xy 154.94 72.39) (xy 154.94 80.01))
+    (stroke (width 0) (type default))
+  )
   (wire (pts (xy 260.35 44.45) (xy 241.3 44.45))
     (stroke (width 0) (type default))
@@
     (stroke (width 0) (type default))
   )
+  (wire (pts (xy 173.99 49.53) (xy 173.99 72.39))
+    (stroke (width 0) (type default))
+  )
   (wire (pts (xy 54.61 133.35) (xy 54.61 139.7))
     (stroke (width 0) (type default))
@@
     (stroke (width 0) (type default))
   )
-  (wire (pts (xy 128.27 72.39) (xy 128.27 80.01))
-    (stroke (width 0) (type default))
-  )
   (wire (pts (xy 106.68 76.2) (xy 137.16 76.2))
     (stroke (width 0) (type default))
@@
     (stroke (width 0) (type default))
   )
-  (wire (pts (xy 128.27 25.4) (xy 186.69 25.4))
-    (stroke (width 0) (type default))
-  )
   (wire (pts (xy 73.66 125.73) (xy 81.28 125.73))
     (stroke (width 0) (type default))
@@
     (stroke (width 0) (type default))
   )
+  (wire (pts (xy 173.99 49.53) (xy 170.18 49.53))
+    (stroke (width 0) (type default))
+  )
+  (wire (pts (xy 170.18 72.39) (xy 154.94 72.39))
+    (stroke (width 0) (type default))
+  )
   (wire (pts (xy 38.1 125.73) (xy 38.1 132.08))
     (stroke (width 0) (type default))
@@
     (stroke (width 0) (type default))
   )
-  (wire (pts (xy 128.27 25.4) (xy 128.27 60.96))
-    (stroke (width 0) (type default))
-  )
   (polyline (pts (xy 12.7 25.4) (xy 12.7 85.09))
     (stroke (width 0) (type default))
   )
-  (wire (pts (xy 170.18 72.39) (xy 154.94 72.39))
+  (wire (pts (xy 173.99 72.39) (xy 170.18 72.39))
     (stroke (width 0) (type default))
   )
@@
     (stroke (width 0) (type default))
   )
-  (wire (pts (xy 128.27 80.01) (xy 208.28 80.01))
+  (wire (pts (xy 99.06 80.01) (xy 154.94 80.01))
     (stroke (width 0) (type default))
   )
@@
   )
   (wire (pts (xy 68.58 125.73) (xy 71.12 125.73))
+    (stroke (width 0) (type default))
+  )
+  (wire (pts (xy 170.18 68.58) (xy 170.18 72.39))
     (stroke (width 0) (type default))
   )
@@
     )
   )
-  (symbol (lib_id "Device:R") (at 128.27 68.58 0) (unit 1)
+  (symbol (lib_id "Device:R") (at 170.18 64.77 0) (unit 1)
     (in_bom yes) (on_board yes) (dnp no) (fields_autoplaced)
-    (property "Reference" "R5" (at 130.81 67.945 0)
-      (effects (font (size 1.27 1.27)) (justify left))
-    )
-    (property "Value" "1k" (at 130.81 70.485 0)
-      (effects (font (size 1.27 1.27)) (justify left))
-    )
-    (property "Footprint" "Resistor_SMD:R_0805_2012Metric_Pad1.20x1.40mm_HandSolder" (at 126.492 68.58 90)
-      (effects (font (size 1.27 1.27)) hide)
-    )
-    (property "Datasheet" "~" (at 128.27 68.58 0)
-      (effects (font (size 1.27 1.27)) hide)
-    )
+    (property "Reference" "R5" (at 172.72 64.135 0)
+      (effects (font (size 1.27 1.27)) (justify left))
+    )
+    (property "Value" "1k" (at 172.72 66.675 0)
+      (effects (font (size 1.27 1.27)) (justify left))
+    )
+    (property "Footprint" "Resistor_SMD:R_0805_2012Metric_Pad1.20x1.40mm_HandSolder" (at 168.402 64.77 90)
+      (effects (font (size 1.27 1.27)) hide)
+    )
+    (property "Datasheet" "~" (at 170.18 64.77 0)
+      (effects (font (size 1.27 1.27)) hide)
+    )
